File: KeyModule-L.kicad_pcb (KiCad board)
At the start: 2 copper layers, 173.5 x 145 mm, 90 parts, among them J1 RJ45, U2 MCP23017

Commit message: update
Other:
- outline, holes or cut-outs redrawn
Changed lines of the file:
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@@
-(kicad_pcb (version 4) (host pcbnew 4.0.2-stable)
+(kicad_pcb (version 4) (host pcbnew 4.0.7)
   (general
     (links 144)
     (no_connects 0)
-    (area 33.911474 11.675 244.714286 166.700001)
+    (area 33.986474 11.825 244.564286 166.700001)
     (thickness 1.6)
     (drawings 442)
@@
     (pad 1 thru_hole circle (at 0 0) (size 3 3) (drill 3) (layers))
   )
+  (gr_line (start 208 16) (end 208 75) (layer Edge.Cuts) (width 0.1))
+  (gr_line (start 208 157) (end 208 75) (layer Edge.Cuts) (width 0.1))
+  (gr_line (start 36.5 159) (end 206 159) (layer Edge.Cuts) (width 0.1))
+  (gr_line (start 34.5 16) (end 34.5 157) (layer Edge.Cuts) (width 0.1))
+  (gr_line (start 206 14) (end 36.5 14) (layer Edge.Cuts) (width 0.1))
   (gr_circle (center 126.5 73.5) (end 126.5 72.5) (layer Eco1.User) (width 0.2))
   (gr_circle (center 118.5 147) (end 118.5 146) (layer Eco1.User) (width 0.2))
@@
     (arrow2b (pts (xy 34.5 164) (xy 35.626504 163.413579)))
   )
-  (gr_line (start 208 14) (end 34.5 14) (layer Edge.Cuts) (width 0.1))
-  (gr_line (start 208 75) (end 208 14) (layer Edge.Cuts) (width 0.1))
-  (gr_line (start 208 159) (end 208 75) (layer Edge.Cuts) (width 0.1))
-  (gr_line (start 34.5 159) (end 208 159) (layer Edge.Cuts) (width 0.1))
-  (gr_line (start 34.5 159) (end 34.5 14) (layer Edge.Cuts) (width 0.1))
   (dimension 145 (width 0.3) (layer Dwgs.User)
     (gr_text "145.000 mm" (at 237.35 86.5 90) (layer Dwgs.User)
