File: _keymodule_l.sch (KiCad schematic (older format))
At the start: 83 parts, among them J1 RJ45, U3 MCP23017

Commit message: footprint
Parts:
- CONBUS1: footprint (none) -> Socket_Strips:Socket_Strip_Straight_1x06
Changed lines of the file:
@@
 LIBS:valves
 LIBS:mylib
-LIBS:Root-cache
+LIBS:KeyModule-L-cache
 EELAYER 25 0
 EELAYER END
 $Descr A3 16535 11693
 encoding utf-8
-Sheet 2 4
+Sheet 2 2
 Title ""
 Date ""
@@
 F 0 "CONBUS1" H 2700 5350 50  0000 C CNN
 F 1 "CONN_01X06" V 2800 5000 50  0000 C CNN
-F 2 "" H 2700 5000 50  0000 C CNN
+F 2 "Socket_Strips:Socket_Strip_Straight_1x06" H 2700 5000 50  0001 C CNN
 F 3 "" H 2700 5000 50  0000 C CNN
 	1    2700 5000
@@
 F 0 "J1" H 3200 7150 50  0000 C CNN
 F 1 "RJ45" H 2850 7150 50  0000 C CNN
-F 2 "" H 3000 6650 50  0000 C CNN
+F 2 "" H 3000 6650 50  0001 C CNN
 F 3 "" H 3000 6650 50  0000 C CNN
 	1    3000 6650

Commit message: update
Parts:
- added BT2, BT3: NiMH1.2V, myfootprint:BAT-P-00308, symbol Battery
- added C1: 0.1u, Capacitors_ThroughHole:C_Rect_L4_W2.5_P2.5, symbol C
- J1: footprint (none) -> myfootprint:RJ45-7810-XPXC
- SW_53, SW_54, SW_55, SW_63, SW_L0, SW_L1, SW_L10, SW_L11, SW_L12, SW_L13, SW_L14, SW_L15, SW_L2, SW_L20, SW_L21, SW_L22, SW_L23, SW_L24, SW_L25, SW_L3, SW_L30, SW_L31, SW_L32, SW_L33, SW_L34, SW_L4, SW_L40, SW_L41, SW_L42, SW_L43, SW_L44, SW_L5, SW_L50, SW_L51, SW_L52, SW_L60, SW_L61, SW_L62, SW_L64, SW_L71: footprint mx1a:MX1A -> myfootprint:MX1A
Connections:
- wire segments 261 -> 266

Commit message: update
Parts:
- BT2, BT3: symbol Battery -> Battery-RESCUE-KeyModule-L
- U3: symbol MCP23017 -> MCP23017-RESCUE-KeyModule-L
Changed lines of the file:
@@
 EESchema Schematic File Version 2
+LIBS:KeyModule-L-rescue
 LIBS:power
 LIBS:device
@@
 LIBS:valves
 LIBS:mylib
-LIBS:Root-cache
+LIBS:KeyModule-L-cache
 EELAYER 25 0
 EELAYER END
 $Descr A3 16535 11693
 encoding utf-8
-Sheet 2 4
+Sheet 2 2
 Title ""
 Date ""
@@
 $EndDescr
 $Comp
-L MCP23017 U3
+L MCP23017-RESCUE-KeyModule-L U3
 U 1 1 5782C5A5
 P 2200 1750
@@
 AR Path="/578B2796/5782C5A5" Ref="U2"  Part="1"
 F 0 "U2" H 2150 850 60  0000 C CNN
-F 1 "MCP23017" H 2100 1750 60  0000 C CNN
+F 1 "MCP23017" H 2000 2750 60  0000 C CNN
 F 2 "Housings_DIP:DIP-28_W7.62mm_LongPads" H 2200 1750 60  0001 C CNN
 F 3 "" H 2200 1750 60  0000 C CNN
@@
 Connection ~ 1150 2050
 $Comp
-L Battery BT2
+L Battery-RESCUE-KeyModule-L BT2
 U 1 1 579CA117
 P 2000 8450
@@
 $EndComp
 $Comp
-L Battery BT3
+L Battery-RESCUE-KeyModule-L BT3
 U 1 1 579CA6BC
 P 2000 8850
