File: _keymodule_r.sch (KiCad schematic (older format))
At the start: 99 parts, among them J2 RJ45, U1 MCP23017

Commit message: footprint
Parts:
- CONBUS2: footprint (none) -> Socket_Strips:Socket_Strip_Straight_1x06
Changed lines of the file:
@@
 LIBS:valves
 LIBS:mylib
-LIBS:Root-cache
+LIBS:KeyModule-R-cache
 EELAYER 25 0
 EELAYER END
 $Descr A3 16535 11693
 encoding utf-8
-Sheet 3 4
+Sheet 3 2
 Title ""
 Date ""
@@
 $EndComp
 $Comp
-L VDD #PWR015
+L VDD #PWR05
 U 1 1 578B9FB2
 P 1250 2300
-F 0 "#PWR015" H 1250 2150 50  0001 C CNN
+F 0 "#PWR05" H 1250 2150 50  0001 C CNN
 F 1 "VDD" H 1250 2450 50  0000 C CNN
 F 2 "" H 1250 2300 50  0000 C CNN
@@
 $EndComp
 $Comp
-L GND #PWR016
+L GND #PWR06
 U 1 1 578B9FB8
 P 1250 2650
-F 0 "#PWR016" H 1250 2400 50  0001 C CNN
+F 0 "#PWR06" H 1250 2400 50  0001 C CNN
 F 1 "GND" H 1250 2500 50  0000 C CNN
 F 2 "" H 1250 2650 50  0000 C CNN
@@
 	3000 2750 4300 2750
 $Comp
-L GND #PWR017
+L GND #PWR07
 U 1 1 578B9FF3
 P 3150 3650
-F 0 "#PWR017" H 3150 3400 50  0001 C CNN
+F 0 "#PWR07" H 3150 3400 50  0001 C CNN
 F 1 "GND" H 3150 3500 50  0000 C CNN
 F 2 "" H 3150 3650 50  0000 C CNN
@@
 $EndComp
 $Comp
-L GND #PWR018
+L GND #PWR08
 U 1 1 578B9FF9
 P 3450 3650
-F 0 "#PWR018" H 3450 3400 50  0001 C CNN
+F 0 "#PWR08" H 3450 3400 50  0001 C CNN
 F 1 "GND" H 3450 3500 50  0000 C CNN
 F 2 "" H 3450 3650 50  0000 C CNN
@@
 $EndComp
 $Comp
-L VDD #PWR019
+L VDD #PWR09
 U 1 1 578BA01A
 P 3950 2900
-F 0 "#PWR019" H 3950 2750 50  0001 C CNN
+F 0 "#PWR09" H 3950 2750 50  0001 C CNN
 F 1 "VDD" H 3950 3050 50  0000 C CNN
 F 2 "" H 3950 2900 50  0000 C CNN
@@
 F 0 "CONBUS2" H 2550 5550 50  0000 C CNN
 F 1 "CONN_01X06" V 2650 5200 50  0000 C CNN
-F 2 "" H 2550 5200 50  0000 C CNN
+F 2 "Socket_Strips:Socket_Strip_Straight_1x06" H 2550 5200 50  0001 C CNN
 F 3 "" H 2550 5200 50  0000 C CNN
 	1    2550 5200
@@
 	2350 5350 2050 5350
 $Comp
-L GND #PWR020
+L GND #PWR010
 U 1 1 57965CC3
 P 2300 5600
-F 0 "#PWR020" H 2300 5350 50  0001 C CNN
+F 0 "#PWR010" H 2300 5350 50  0001 C CNN
 F 1 "GND" H 2300 5450 50  0000 C CNN
 F 2 "" H 2300 5600 50  0000 C CNN
@@
 $EndComp
 $Comp
-L VDD #PWR021
+L VDD #PWR011
 U 1 1 57965CC9
 P 2300 4850
-F 0 "#PWR021" H 2300 4700 50  0001 C CNN
+F 0 "#PWR011" H 2300 4700 50  0001 C CNN
 F 1 "VDD" H 2300 5000 50  0000 C CNN
 F 2 "" H 2300 4850 50  0000 C CNN
@@
 F 0 "J2" H 3050 7350 50  0000 C CNN
 F 1 "RJ45" H 2700 7350 50  0000 C CNN
-F 2 "" H 2850 6850 50  0000 C CNN
+F 2 "" H 2850 6850 50  0001 C CNN
 F 3 "" H 2850 6850 50  0000 C CNN
 	1    2850 6850
@@
 $EndComp
 $Comp
-L GND #PWR022
+L GND #PWR012
 U 1 1 57965CDA
 P 2300 7300
-F 0 "#PWR022" H 2300 7050 50  0001 C CNN
+F 0 "#PWR012" H 2300 7050 50  0001 C CNN
 F 1 "GND" H 2300 7150 50  0000 C CNN
 F 2 "" H 2300 7300 50  0000 C CNN
@@
 $EndComp
 $Comp
-L VDD #PWR023
+L VDD #PWR013
 U 1 1 57965CE0
 P 2300 6250
-F 0 "#PWR023" H 2300 6100 50  0001 C CNN
+F 0 "#PWR013" H 2300 6100 50  0001 C CNN
 F 1 "VDD" H 2300 6400 50  0000 C CNN
 F 2 "" H 2300 6250 50  0000 C CNN
@@
 Connection ~ 2300 7200
 $Comp
-L GND #PWR024
+L GND #PWR014
 U 1 1 57965CEE
 P 3200 7400
-F 0 "#PWR024" H 3200 7150 50  0001 C CNN
+F 0 "#PWR014" H 3200 7150 50  0001 C CNN
 F 1 "GND" H 3200 7250 50  0000 C CNN
 F 2 "" H 3200 7400 50  0000 C CNN

Commit message: update
Parts:
- added BT4, BT5: NiMH1.2V, myfootprint:BAT-P-00308, symbol Battery
- added C2: 0.1u, Capacitors_ThroughHole:C_Rect_L4_W2.5_P2.5, symbol C
- J2: footprint (none) -> myfootprint:RJ45-7810-XPXC
- SW_64, SW_R1, SW_R10, SW_R11, SW_R12, SW_R13, SW_R14, SW_R15, SW_R16, SW_R2, SW_R20, SW_R21, SW_R22, SW_R23, SW_R24, SW_R25, SW_R26, SW_R3, SW_R30, SW_R31, SW_R32, SW_R33, SW_R34, SW_R4, SW_R40, SW_R41, SW_R42, SW_R43, SW_R44, SW_R45, SW_R50, SW_R51, SW_R52, SW_R53, SW_R54, SW_R55, SW_R6, SW_R60, SW_R61, SW_R62, SW_R63, SW_R65, SW_R70, SW_R71, SW_R72, SW_R73, SW_R74, SW_R75: footprint mx1a:MX1A -> myfootprint:MX1A
Connections:
- wire segments 302 -> 307

Commit message: update
Parts:
- BT4, BT5: symbol Battery -> Battery-RESCUE-KeyModule-R
- U1: symbol MCP23017 -> MCP23017-RESCUE-KeyModule-R
Changed lines of the file:
@@
 EESchema Schematic File Version 2
+LIBS:KeyModule-R-rescue
 LIBS:power
 LIBS:device
@@
 LIBS:valves
 LIBS:mylib
-LIBS:Root-cache
+LIBS:KeyModule-R-cache
 EELAYER 25 0
 EELAYER END
 $Descr A3 16535 11693
 encoding utf-8
-Sheet 3 4
+Sheet 3 2
 Title ""
 Date ""
@@
 $EndDescr
 $Comp
-L MCP23017 U1
+L MCP23017-RESCUE-KeyModule-R U1
 U 1 1 578B9FAB
 P 2450 2000
@@
 	1600 2450 1600 2300
 $Comp
-L Battery BT4
+L Battery-RESCUE-KeyModule-R BT4
 U 1 1 579CB558
 P 2150 8950
@@
 $EndComp
 $Comp
-L Battery BT5
+L Battery-RESCUE-KeyModule-R BT5
 U 1 1 579CB55F
 P 2150 9350
