File: _main.sch (KiCad schematic (older format))
At the start: 12 parts, among them P1 CONN_01X06, U3 BLE_NANO

Commit message: footprint
Parts:
- P1: footprint (none) -> Pin_Headers:Pin_Header_Straight_1x06
- P_GND1, P_RXD1, P_SWCLK1, P_SWDIO1, P_TXD1: footprint (none) -> Socket_Strips:Socket_Strip_Straight_1x01
- R1, R2, R3: footprint Resistors_SMD:R_0603_HandSoldering -> Resistors_ThroughHole:Resistor_Horizontal_RM7mm
Changed lines of the file:
@@
 LIBS:valves
 LIBS:mylib
-LIBS:Root-cache
+LIBS:Main-cache
 EELAYER 25 0
 EELAYER END
 $Descr A4 11693 8268
 encoding utf-8
-Sheet 4 4
+Sheet 4 2
 Title ""
 Date ""
@@
 F 0 "P1" H 6800 5250 50  0000 C CNN
 F 1 "CONN_01X06" V 6900 4900 50  0000 C CNN
-F 2 "" H 6800 4900 50  0000 C CNN
+F 2 "Pin_Headers:Pin_Header_Straight_1x06" H 6800 4900 50  0001 C CNN
 F 3 "" H 6800 4900 50  0000 C CNN
 	1    6800 4900
@@
 	6300 5050 6600 5050
 $Comp
-L GND #PWR025
+L GND #PWR05
 U 1 1 579615BF
 P 6550 5300
-F 0 "#PWR025" H 6550 5050 50  0001 C CNN
+F 0 "#PWR05" H 6550 5050 50  0001 C CNN
 F 1 "GND" H 6550 5150 50  0000 C CNN
 F 2 "" H 6550 5300 50  0000 C CNN
@@
 $EndComp
 $Comp
-L VDD #PWR026
+L VDD #PWR06
 U 1 1 579615C5
 P 6550 4550
-F 0 "#PWR026" H 6550 4400 50  0001 C CNN
+F 0 "#PWR06" H 6550 4400 50  0001 C CNN
 F 1 "VDD" H 6550 4700 50  0000 C CNN
 F 2 "" H 6550 4550 50  0000 C CNN
@@
 	6550 5150 6550 5300
 $Comp
-L GND #PWR027
+L GND #PWR07
 U 1 1 579617D8
 P 4200 2650
-F 0 "#PWR027" H 4200 2400 50  0001 C CNN
+F 0 "#PWR07" H 4200 2400 50  0001 C CNN
 F 1 "GND" H 4200 2500 50  0000 C CNN
 F 2 "" H 4200 2650 50  0000 C CNN
@@
 NoConn ~ 4400 2500
 $Comp
-L VDD #PWR028
+L VDD #PWR08
 U 1 1 579617DF
 P 6450 1500
-F 0 "#PWR028" H 6450 1350 50  0001 C CNN
+F 0 "#PWR08" H 6450 1350 50  0001 C CNN
 F 1 "VDD" H 6450 1650 50  0000 C CNN
 F 2 "" H 6450 1500 50  0000 C CNN
@@
 $EndComp
 $Comp
-L GND #PWR029
+L GND #PWR09
 U 1 1 579617E5
 P 6450 2650
-F 0 "#PWR029" H 6450 2400 50  0001 C CNN
+F 0 "#PWR09" H 6450 2400 50  0001 C CNN
 F 1 "GND" H 6450 2500 50  0000 C CNN
 F 2 "" H 6450 2650 50  0000 C CNN
@@
 F 0 "R1" V 3530 2450 50  0000 C CNN
 F 1 "10" V 3450 2450 50  0000 C CNN
-F 2 "Resistors_SMD:R_0603_HandSoldering" V 3380 2450 50  0001 C CNN
+F 2 "Resistors_ThroughHole:Resistor_Horizontal_RM7mm" V 3380 2450 50  0001 C CNN
 F 3 "" H 3450 2450 50  0000 C CNN
 	1    3450 2450
@@
 $EndComp
 $Comp
-L GND #PWR030
+L GND #PWR010
 U 1 1 57961800
 P 3450 3200
-F 0 "#PWR030" H 3450 2950 50  0001 C CNN
+F 0 "#PWR010" H 3450 2950 50  0001 C CNN
 F 1 "GND" H 3450 3050 50  0000 C CNN
 F 2 "" H 3450 3200 50  0000 C CNN
@@
 	3450 3150 3450 3200
 $Comp
-L VDD #PWR031
+L VDD #PWR011
 U 1 1 57961813
 P 8300 1450
-F 0 "#PWR031" H 8300 1300 50  0001 C CNN
+F 0 "#PWR011" H 8300 1300 50  0001 C CNN
 F 1 "VDD" H 8300 1600 50  0000 C CNN
 F 2 "" H 8300 1450 50  0000 C CNN
@@
 RXD
 $Comp
-L VDD #PWR032
+L VDD #PWR012
 U 1 1 57961828
 P 6900 1500
-F 0 "#PWR032" H 6900 1350 50  0001 C CNN
+F 0 "#PWR012" H 6900 1350 50  0001 C CNN
 F 1 "VDD" H 6900 1650 50  0000 C CNN
 F 2 "" H 6900 1500 50  0000 C CNN
@@
 F 0 "R2" V 6980 1800 50  0000 C CNN
 F 1 "10k" V 6900 1800 50  0000 C CNN
-F 2 "Resistors_SMD:R_0603_HandSoldering" V 6830 1800 50  0001 C CNN
+F 2 "Resistors_ThroughHole:Resistor_Horizontal_RM7mm" V 6830 1800 50  0001 C CNN
 F 3 "" H 6900 1800 50  0000 C CNN
 	1    6900 1800
@@
 F 0 "R3" V 7180 1800 50  0000 C CNN
 F 1 "10k" V 7100 1800 50  0000 C CNN
-F 2 "Resistors_SMD:R_0603_HandSoldering" V 7030 1800 50  0001 C CNN
+F 2 "Resistors_ThroughHole:Resistor_Horizontal_RM7mm" V 7030 1800 50  0001 C CNN
 F 3 "" H 7100 1800 50  0000 C CNN
 	1    7100 1800
@@
 F 0 "P_SWCLK1" H 1700 3200 50  0000 C CNN
 F 1 "CONN_01X01" V 1800 3100 50  0001 C CNN
-F 2 "" H 1700 3100 50  0000 C CNN
+F 2 "Socket_Strips:Socket_Strip_Straight_1x01" H 1700 3100 50  0001 C CNN
 F 3 "" H 1700 3100 50  0000 C CNN
 	1    1700 3100
@@
 F 0 "P_SWDIO1" H 1700 3450 50  0000 C CNN
 F 1 "CONN_01X01" V 1800 3350 50  0001 C CNN
-F 2 "" H 1700 3350 50  0000 C CNN
+F 2 "Socket_Strips:Socket_Strip_Straight_1x01" H 1700 3350 50  0001 C CNN
 F 3 "" H 1700 3350 50  0000 C CNN
 	1    1700 3350
@@
 F 0 "P_GND1" H 1700 3700 50  0000 C CNN
 F 1 "CONN_01X01" V 1800 3600 50  0001 C CNN
-F 2 "" H 1700 3600 50  0000 C CNN
+F 2 "Socket_Strips:Socket_Strip_Straight_1x01" H 1700 3600 50  0001 C CNN
 F 3 "" H 1700 3600 50  0000 C CNN
 	1    1700 3600
@@
 F 0 "P_TXD1" H 1700 3950 50  0000 C CNN
 F 1 "CONN_01X01" V 1800 3850 50  0001 C CNN
-F 2 "" H 1700 3850 50  0000 C CNN
+F 2 "Socket_Strips:Socket_Strip_Straight_1x01" H 1700 3850 50  0001 C CNN
 F 3 "" H 1700 3850 50  0000 C CNN
 	1    1700 3850
@@
 F 0 "P_RXD1" H 1700 4200 50  0000 C CNN
 F 1 "CONN_01X01" V 1800 4100 50  0001 C CNN
-F 2 "" H 1700 4100 50  0000 C CNN
+F 2 "Socket_Strips:Socket_Strip_Straight_1x01" H 1700 4100 50  0001 C CNN
 F 3 "" H 1700 4100 50  0000 C CNN
 	1    1700 4100
@@
 $EndComp
 $Comp
-L GND #PWR033
+L GND #PWR013
 U 1 1 57961B4E
 P 2700 5450
-F 0 "#PWR033" H 2700 5200 50  0001 C CNN
+F 0 "#PWR013" H 2700 5200 50  0001 C CNN
 F 1 "GND" H 2700 5300 50  0000 C CNN
 F 2 "" H 2700 5450 50  0000 C CNN
@@
 $EndComp
 $Comp
-L VDD #PWR034
+L VDD #PWR014
 U 1 1 57961B54
 P 2700 4900
-F 0 "#PWR034" H 2700 4750 50  0001 C CNN
+F 0 "#PWR014" H 2700 4750 50  0001 C CNN
 F 1 "VDD" H 2700 5050 50  0000 C CNN
 F 2 "" H 2700 4900 50  0000 C CNN

Commit message: update
Parts:
- added P_GND2: CONN_01X01, Socket_Strips:Socket_Strip_Straight_1x01, symbol CONN_01X01
- added SW1: SW_RESET, Buttons_Switches_ThroughHole:SW_PUSH-12mm, symbol SW_PUSH
- R1: value 10 -> 4.7k
Connections:
- wire segments 30 -> 34
Other:
- moved on the sheet: P_GND1
Changed lines of the file:
@@
 $Descr A4 11693 8268
 encoding utf-8
-Sheet 4 2
+Sheet 2 2
 Title ""
 Date ""
@@
 P 3450 2450
 F 0 "R1" V 3530 2450 50  0000 C CNN
-F 1 "10" V 3450 2450 50  0000 C CNN
+F 1 "4.7k" V 3450 2450 50  0000 C CNN
 F 2 "Resistors_ThroughHole:Resistor_Horizontal_RM7mm" V 3380 2450 50  0001 C CNN
 F 3 "" H 3450 2450 50  0000 C CNN
@@
 L CONN_01X01 P_GND1
 U 1 1 579619D9
-P 1700 3600
-F 0 "P_GND1" H 1700 3700 50  0000 C CNN
-F 1 "CONN_01X01" V 1800 3600 50  0001 C CNN
-F 2 "Socket_Strips:Socket_Strip_Straight_1x01" H 1700 3600 50  0001 C CNN
-F 3 "" H 1700 3600 50  0000 C CNN
-	1    1700 3600
+P 2450 3100
+F 0 "P_GND1" H 2450 3200 50  0000 C CNN
+F 1 "CONN_01X01" V 2550 3100 50  0001 C CNN
+F 2 "Socket_Strips:Socket_Strip_Straight_1x01" H 2450 3100 50  0001 C CNN
+F 3 "" H 2450 3100 50  0000 C CNN
+	1    2450 3100
 	-1   0    0    1
 $EndComp
@@
 Text Label 1900 3350 0    60   ~ 0
 SWDIO
-Text Label 1900 3600 0    60   ~ 0
+Text Label 2650 3100 0    60   ~ 0
 GND
 Text Label 1900 3850 0    60   ~ 0
@@
 Text GLabel 6300 5050 0    60   Input ~ 0
 INT
+$Comp
+L SW_PUSH SW1
+U 1 1 57BF185A
+P 3700 1500
+F 0 "SW1" H 3850 1610 50  0000 C CNN
+F 1 "SW_RESET" H 3700 1420 50  0000 C CNN
+F 2 "Buttons_Switches_ThroughHole:SW_PUSH-12mm" H 3700 1500 50  0001 C CNN
+F 3 "" H 3700 1500 50  0000 C CNN
+	1    3700 1500
+	1    0    0    -1
+$EndComp
+$Comp
+L GND #PWR015
+U 1 1 57BF197C
+P 3400 1700
+F 0 "#PWR015" H 3400 1450 50  0001 C CNN
+F 1 "GND" H 3400 1550 50  0000 C CNN
+F 2 "" H 3400 1700 50  0000 C CNN
+F 3 "" H 3400 1700 50  0000 C CNN
+	1    3400 1700
+	1    0    0    -1
+$EndComp
+Wire Wire Line
+	4400 2100 4050 2100
+Wire Wire Line
+	4050 2100 4050 1500
+Wire Wire Line
+	4050 1500 4000 1500
+Wire Wire Line
+	3400 1500 3400 1700
+$Comp
+L CONN_01X01 P_GND2
+U 1 1 57C199FB
+P 2350 3850
+F 0 "P_GND2" H 2350 3950 50  0000 C CNN
+F 1 "CONN_01X01" V 2450 3850 50  0001 C CNN
+F 2 "Socket_Strips:Socket_Strip_Straight_1x01" H 2350 3850 50  0001 C CNN
+F 3 "" H 2350 3850 50  0000 C CNN
+	1    2350 3850
+	-1   0    0    1
+$EndComp
+Text Label 2550 3850 0    60   ~ 0
+GND
 $EndSCHEMATC

Commit message: update
Parts:
- BT1: symbol Battery -> Battery-RESCUE-Main
- D1: symbol LED -> LED-RESCUE-Main
Changed lines of the file:
@@
 EESchema Schematic File Version 2
+LIBS:Main-rescue
 LIBS:power
 LIBS:device
@@
 NoConn ~ 5450 3300
 $Comp
-L LED D1
+L LED-RESCUE-Main D1
 U 1 1 579617F2
 P 3450 2950
@@
 RXD
 $Comp
-L Battery BT1
+L Battery-RESCUE-Main BT1
 U 1 1 57961B47
 P 2700 5200
